File: FWBR_PCB_Design/FWBR_PCB_Design.kicad_sch (KiCad schematic)
At the start: 0 parts

Commit message: Lt Spice stuff
Parts:
- added C1: C_Polarized, symbol Device:C_Polarized
- added C2: 1u, symbol Device:C
- added C3: 10n, symbol Device:C
- added C4, C5: C, symbol Device:C
- added C6: 0.1u, symbol Device:C
- added D1, D2, D3, D4: PMEG6010ELR, Diode_SMD:Nexperia_CFP3_SOD-123W, symbol Diode:PMEG6010ELR
- added J1: Screw_Terminal_01x02, symbol Connector:Screw_Terminal_01x02
- added L1: L, symbol Device:L
- added R1, R2, R3, R4: R, symbol Device:R
- added U1: LT8606IMSE-PBF, MSE_10_ADI, symbol 2026-08-05_22-53-31:LT8606IMSE-PBF
Connections:
- new net: C6.1, L1.1, U1.2 (SW)
- new net: C3.1, U1.7 (TR/SS)
- new net: C1.1, D2.1 (K), D4.1 (K)
- new net: D3.1 (K), D4.2 (A), J1.2 (Pin_2)
- new net: C6.2, U1.1 (BST)
- new net: R3.1, R4.2, U1.10 (EN/UV)
- new net: C2.1, U1.3 (INTVCC)
- new net: C4.1, C4.2, C5.1, R1.1, R1.2, R2.1, U1.6 (FB)
- new net: R3.2, U1.9 (VIN)
- new net: D1.1 (K), D2.2 (A), J1.1 (Pin_1)
- new net GND: C1.2, C2.2, C3.2, C5.2, D1.2 (A), D3.2 (A), R2.2, R4.1, U1.EPAD
